File: HardwareDesign.kicad_sch (KiCad schematic)
At the start: 1 part

Commit message: Initial Draft of Test Board
Parts:
- removed D1: QCA 7000, Package_DFN_QFN:QFN-68-1EP_8x8mm_P0.4mm_EP5.2x5.2mm_ThermalVias, symbol QualcommAtheros:QCA 7000
Other:
- added sheet Control Pilot (CP.kicad_sch)
- added sheet ESP32 (controller.kicad_sch)
- added sheet Power (Power.kicad_sch)
- added sheet QCA7000 (QCA7000.kicad_sch)
