File: HardwareDesign.kicad_pcb (KiCad board)
At the start: 2 copper layers, 130 x 130 mm, 271 parts, among them J1 Conn_01x07, J2 U263-163N-4BQC65, J3 Conn_02x03_Odd_Even, J4 Conn_01x07, J5 Screw_Terminal_01x03, Q1 SI2323DS, T1 CL4532A-201, U1 W25Q128JVS, U10 AMS1117-ADJ, U11 OPA2991IDR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

Commit message: 1st test board manufacturing files
Parts:
- D4, D5, D6, D7: value 1N5819 -> B5819W SL
- R22: footprint Resistor_SMD:R_0805_2012Metric -> Resistor_SMD:R_0603_1608Metric
- moved J5 24.6 mm to (150.6, 143.2)
- moved T1 1.75 mm to (135.7, 130.5)
- moved C98 1.75 mm to (122.4, 133.7)
- moved C97 1.75 mm to (136.8, 136.2)
- moved D16 1.75 mm to (125.8, 131.7)
- moved R37 1.75 mm to (136.8, 134.0)
- moved R22 0.13 mm to (96.3, 88.8)
Connections:
- C10 pad 2: Net-(C10-Pad2) -> GND
- C11 pad 1: Net-(C10-Pad2) -> GND
- C3 pad 2: Net-(C3-Pad2) -> GND
- C38 pad 1: Net-(D6-K) -> GND
- C38 pad 2: Net-(C38-Pad2) -> Net-(D6-K)
- C4 pad 1: Net-(C3-Pad2) -> GND
- L1 pad 2: Net-(L1-Pad2) -> GND
- L2 pad 1: Net-(L1-Pad2) -> GND
- L5 pad 2: Net-(L5-Pad2) -> GND
- L6 pad 1: Net-(L5-Pad2) -> GND
- L9 pad 1: Net-(C38-Pad2) -> Net-(D6-K)
Routing:
- net CP_OUT: track 69.9 -> 91.4 mm
- net GND: track 161.3 -> 171.7 mm, vias 133 -> 136
- net Net-(D6-K): track 10.2 -> 14.6 mm
- net Net-(C3-Pad2): track 1.90 -> 0.00 mm
- net Net-(C10-Pad2): track 1.80 -> 0.00 mm
- net Net-(C38-Pad2): track 1.80 -> 0.00 mm
- net RX_N: track 20.0 -> 21.7 mm
- net TX_P: track 7.66 -> 5.92 mm
- net TX_N: track 7.92 -> 6.19 mm
- net RX_P: track 13.5 -> 15.2 mm
- net Net-(L5-Pad2): track 1.58 -> 0.00 mm
- net Net-(L1-Pad2): track 1.58 -> 0.00 mm
