File: QCA7000.kicad_sch (KiCad schematic)
At the start: 122 parts, among them J1 Conn_01x07, T1 CL4532A-201, U1 W25Q128JVS, Y1 25MHz

Commit message: 1st test board manufacturing files
Parts:
- D4, D5, D6, D7: value 1N5819 -> B5819W SL
- J1: JLCPCB Part No # C6332200 -> (none)
- L9: value L_Ferrite -> GZ2012D601TF
- Y1: value 25MHz -> 25MHz X322525MOB4SI
Connections:
- net GND: now also C10.2, C11.1, C3.2, C38.1, C4.1, L1.2, L2.1, L5.2, L6.1
- net at C38.2, L9.1: now also C36.2, D6.1 (K), D7.1 (K), D8.1 (K)
Other:
- moved on the sheet: C38
