File: controller.kicad_sch (KiCad schematic)
At the start: 30 parts, among them J2 U263-163N-4BQC65, J3 Conn_02x03_Odd_Even, J4 Conn_01x07, U2 ESP32-S3-WROOM-1

Commit message: 1st test board manufacturing files
Parts:
- J3: value Conn_02x03_Odd_Even -> HC-JN254-2-03-Z
Changed lines of the file:
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@@
 			)
 		)
-		(property "Value" "Conn_02x03_Odd_Even"
+		(property "Value" "HC-JN254-2-03-Z"
 			(at 245.11 71.12 0)
 			(effects
